File: keyboard.kicad_pcb (KiCad board)
At the start: 2 copper layers, 24 parts, among them SW1 RESET, U1 ATmega32U4-A, Y1 16MHz

Commit message: Fixed errors + gerber files
Routing:
- added copper zone on B.Cu, net GND
Other:
- board outline added: 72.2 x 38.1 mm
Changed lines of the file:
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@@
     (pad_to_mask_clearance 0)
     (pcbplotparams
-      (layerselection 0x00010fc_ffffffff)
+      (layerselection 0x00010f0_ffffffff)
       (plot_on_all_layers_selection 0x0000000_00000000)
       (disableapertmacros false)
@@
       (outputformat 1)
       (mirror false)
-      (drillshape 1)
+      (drillshape 0)
       (scaleselection 1)
       (outputdirectory "")
@@
     (fp_line (start 1 0.625) (end 1 -0.625)
       (stroke (width 0.1) (type solid)) (layer "B.Fab"))
-    (pad "1" smd roundrect (at -0.9125 0 180) (size 1.025 1.4) (layers "B.Cu" "B.Paste" "B.Mask") (roundrect_rratio 0.243902)
+    (pad "1" smd roundrect (at -0.9125 0 180) (size 1.025 1.4) (layers "B.Cu" "B.Paste" "B.Mask") (roundrect_rratio 0.243902439)
       (net 18 "D-") (pintype "passive"))
-    (pad "2" smd roundrect (at 0.9125 0 180) (size 1.025 1.4) (layers "B.Cu" "B.Paste" "B.Mask") (roundrect_rratio 0.243902)
+    (pad "2" smd roundrect (at 0.9125 0 180) (size 1.025 1.4) (layers "B.Cu" "B.Paste" "B.Mask") (roundrect_rratio 0.243902439)
       (net 19 "Net-(U1-D-)") (pintype "passive"))
     (model "${KICAD6_3DMODEL_DIR}/Resistor_SMD.3dshapes/R_0805_2012Metric.wrl"
@@
     (fp_line (start 1 0.625) (end 1 -0.625)
       (stroke (width 0.1) (type solid)) (layer "B.Fab"))
-    (pad "1" smd roundrect (at -0.9125 0 180) (size 1.025 1.4) (layers "B.Cu" "B.Paste" "B.Mask") (roundrect_rratio 0.243902)
+    (pad "1" smd roundrect (at -0.9125 0 180) (size 1.025 1.4) (layers "B.Cu" "B.Paste" "B.Mask") (roundrect_rratio 0.243902439)
       (net 16 "D+") (pintype "passive"))
-    (pad "2" smd roundrect (at 0.9125 0 180) (size 1.025 1.4) (layers "B.Cu" "B.Paste" "B.Mask") (roundrect_rratio 0.243902)
+    (pad "2" smd roundrect (at 0.9125 0 180) (size 1.025 1.4) (layers "B.Cu" "B.Paste" "B.Mask") (roundrect_rratio 0.243902439)
       (net 17 "Net-(U1-D+)") (pintype "passive"))
     (model "${KICAD6_3DMODEL_DIR}/Resistor_SMD.3dshapes/R_0805_2012Metric.wrl"
@@
     (fp_line (start 1 0.625) (end 1 -0.625)
       (stroke (width 0.1) (type solid)) (layer "B.Fab"))
-    (pad "1" smd roundrect (at -0.9125 0) (size 1.025 1.4) (layers "B.Cu" "B.Paste" "B.Mask") (roundrect_rratio 0.243902)
+    (pad "1" smd roundrect (at -0.9125 0) (size 1.025 1.4) (layers "B.Cu" "B.Paste" "B.Mask") (roundrect_rratio 0.243902439)
       (net 5 "+5V") (pintype "passive"))
-    (pad "2" smd roundrect (at 0.9125 0) (size 1.025 1.4) (layers "B.Cu" "B.Paste" "B.Mask") (roundrect_rratio 0.243902)
+    (pad "2" smd roundrect (at 0.9125 0) (size 1.025 1.4) (layers "B.Cu" "B.Paste" "B.Mask") (roundrect_rratio 0.243902439)
       (net 15 "Net-(U1-~{RESET})") (pintype "passive"))
     (model "${KICAD6_3DMODEL_DIR}/Resistor_SMD.3dshapes/R_0805_2012Metric.wrl"
@@
     (fp_line (start 1 0.625) (end 1 -0.625)
       (stroke (width 0.1) (type solid)) (layer "B.Fab"))
-    (pad "1" smd roundrect (at -0.9125 0 90) (size 1.025 1.4) (layers "B.Cu" "B.Paste" "B.Mask") (roundrect_rratio 0.243902)
+    (pad "1" smd roundrect (at -0.9125 0 90) (size 1.025 1.4) (layers "B.Cu" "B.Paste" "B.Mask") (roundrect_rratio 0.243902439)
       (net 20 "Net-(U1-~{HWB}{slash}PE2)") (pintype "passive"))
-    (pad "2" smd roundrect (at 0.9125 0 90) (size 1.025 1.4) (layers "B.Cu" "B.Paste" "B.Mask") (roundrect_rratio 0.243902)
+    (pad "2" smd roundrect (at 0.9125 0 90) (size 1.025 1.4) (layers "B.Cu" "B.Paste" "B.Mask") (roundrect_rratio 0.243902439)
       (net 2 "GND") (pintype "passive"))
     (model "${KICAD6_3DMODEL_DIR}/Resistor_SMD.3dshapes/R_0805_2012Metric.wrl"
@@
     )
   )
+  (gr_line (start 105.56875 93.6625) (end 173.0375 93.6625)
+    (stroke (width 0.1) (type default)) (layer "Edge.Cuts"))
+  (gr_arc (start 105.56875 93.6625) (mid 103.884952 92.965048) (end 103.1875 91.28125)
+    (stroke (width 0.1) (type default)) (layer "Edge.Cuts"))
   (gr_arc (start 103.1875 57.94375) (mid 103.884952 56.259952) (end 105.56875 55.5625)
-    (stroke (width 0.2) (type default)) (layer "F.Cu"))
-  (gr_line (start 105.56875 93.6625) (end 173.0375 93.6625)
-    (stroke (width 0.2) (type default)) (layer "F.Cu"))
-  (gr_line (start 175.41875 57.94375) (end 175.41875 91.28125)
-    (stroke (width 0.2) (type default)) (layer "F.Cu"))
+    (stroke (width 0.1) (type default)) (layer "Edge.Cuts"))
+  (gr_arc (start 175.41875 91.28125) (mid 174.721298 92.965048) (end 173.0375 93.6625)
+    (stroke (width 0.1) (type default)) (layer "Edge.Cuts"))
   (gr_line (start 103.1875 57.94375) (end 103.1875 91.28125)
-    (stroke (width 0.2) (type default)) (layer "F.Cu"))
+    (stroke (width 0.1) (type default)) (layer "Edge.Cuts"))
+  (gr_line (start 175.41875 91.28125) (end 175.41875 57.94375)
+    (stroke (width 0.1) (type default)) (layer "Edge.Cuts"))
   (gr_line (start 173.0375 55.5625) (end 105.56875 55.5625)
-    (stroke (width 0.2) (type default)) (layer "F.Cu"))
+    (stroke (width 0.1) (type default)) (layer "Edge.Cuts"))
   (gr_arc (start 173.0375 55.5625) (mid 174.721298 56.259952) (end 175.41875 57.94375)
-    (stroke (width 0.2) (type default)) (layer "F.Cu"))
-  (gr_arc (start 105.56875 93.6625) (mid 103.884952 92.965048) (end 103.1875 91.28125)
-    (stroke (width 0.2) (type default)) (layer "F.Cu"))
+    (stroke (width 0.1) (type default)) (layer "Edge.Cuts"))
   (segment (start 155.52925 79.32925) (end 155.52925 77.83525) (width 0.254) (layer "B.Cu") (net 1))
   (segment (start 148.12225 81.34525) (end 144.86125 81.34525) (width 0.254) (layer "B.Cu") (net 1))
@@
   (segment (start 147.79625 68.04025) (end 149.73425 68.04025) (width 0.254) (layer "B.Cu") (net 20))
   (segment (start 149.73425 68.04025) (end 149.82925 68.13525) (width 0.254) (layer "B.Cu") (net 20))
+  (zone (net 2) (net_name "GND") (layer "B.Cu") (hatch edge 0.5)
+    (connect_pads (clearance 0.5))
+    (min_thickness 0.25) (filled_areas_thickness no)
+    (fill yes (thermal_gap 0.5) (thermal_bridge_width 0.5))
+    (polygon
+      (pts
+        (xy 141.2875 55.5625)
+        (xy 141.2875 93.6625)
+        (xy 175.41875 93.6625)
+        (xy 175.41875 55.5625)
+      )
+    )
+  )
 )
